File: pro_tiny.kicad_sch (KiCad schematic)
At the start: 24 parts, among them J1 Conn_01x12, J2 Conn_01x12, J3 Conn_01x04, J4 USB_C_Receptacle_USB2.0, U1 ATmega32U4-M, Y1 16mhz

Commit message: finished routing main pins
Parts:
- D1: footprint Diode_SMD:D_0603_1608Metric -> Diode_SMD:D_0402_1005Metric
Connections:
- net VBUS is gone; now on net +5V: C1.1, J4.A4 (VBUS), J4.A9 (VBUS), J4.B4 (VBUS), J4.B9 (VBUS), R3.2, U1.7 (VBUS)
Changed lines of the file:
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@@
   (junction (at 165.1 40.64) (diameter 0) (color 0 0 0 0)
   )
+  (junction (at 43.18 60.96) (diameter 0) (color 0 0 0 0)
+  )
   (junction (at 170.18 40.64) (diameter 0) (color 0 0 0 0)
   )
@@
     (stroke (width 0) (type default) (color 0 0 0 0))
   )
+  (wire (pts (xy 43.18 60.96) (xy 45.72 60.96))
+    (stroke (width 0) (type default) (color 0 0 0 0))
+  )
   (wire (pts (xy 19.05 45.72) (xy 19.05 48.26))
     (stroke (width 0) (type default) (color 0 0 0 0))
@@
     (stroke (width 0) (type default) (color 0 0 0 0))
   )
+  (wire (pts (xy 43.18 59.69) (xy 43.18 60.96))
+    (stroke (width 0) (type default) (color 0 0 0 0))
+  )
   (wire (pts (xy 76.2 71.12) (xy 77.47 71.12))
     (stroke (width 0) (type default) (color 0 0 0 0))
@@
     (stroke (width 0) (type default) (color 0 0 0 0))
   )
-  (wire (pts (xy 40.64 60.96) (xy 45.72 60.96))
+  (wire (pts (xy 40.64 60.96) (xy 43.18 60.96))
     (stroke (width 0) (type default) (color 0 0 0 0))
   )
@@
     (pin "1")
     (pin "2")
+  )
+  (symbol (lib_id "power:+5V") (at 43.18 59.69 0) (unit 1)
+    (in_bom yes) (on_board yes)
+    (property "Reference" "#PWR?" (id 0) (at 43.18 63.5 0)
+      (effects (font (size 1.27 1.27)) hide)
+    )
+    (property "Value" "+5V" (id 1) (at 39.37 58.42 0))
+    (property "Footprint" "" (id 2) (at 43.18 59.69 0)
+      (effects (font (size 1.27 1.27)) hide)
+    )
+    (property "Datasheet" "" (id 3) (at 43.18 59.69 0)
+      (effects (font (size 1.27 1.27)) hide)
+    )
+    (pin "1")
   )
   (symbol (lib_id "power:GND") (at 40.64 83.82 0) (unit 1)
@@
       (effects (font (size 1.27 1.27)) (justify left))
     )
-    (property "Footprint" "Diode_SMD:D_0603_1608Metric" (id 2) (at 26.67 29.21 90)
+    (property "Footprint" "Diode_SMD:D_0402_1005Metric" (id 2) (at 26.67 29.21 90)
       (effects (font (size 1.27 1.27)) hide)
     )
@@
       (reference "#PWR0117") (unit 1) (value "GND") (footprint "")
     )
+    (path "/a8a0b327-3339-47b9-9b64-64aafed91f6b"
+      (reference "#PWR?") (unit 1) (value "+5V") (footprint "")
+    )
     (path "/fea89e33-8ea8-4159-b2ab-9301a5e5d74d"
       (reference "C1") (unit 1) (value "100nf") (footprint "Capacitor_SMD:C_0402_1005Metric")
@@
     )
     (path "/e7416661-ba9b-499d-8603-5221b2873cf5"
-      (reference "D1") (unit 1) (value "D_Small") (footprint "Diode_SMD:D_0603_1608Metric")
+      (reference "D1") (unit 1) (value "D_Small") (footprint "Diode_SMD:D_0402_1005Metric")
     )
     (path "/2bf7c2a7-1ea3-4592-a226-b942f45a6bdb"
