File: epi.kicad_sch (KiCad schematic)
At the start: 28 parts, among them J1 Connector 1x12, J2 Connector 1x12, J3 Conn_01x05, J4 USB-C 2.0 mid-mount female co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, U1 ATmega32U4-M, Y1 Crystal_GND24_Small

Commit message: bit of everything
Parts:
- added TP1, TP2: TestPoint, TestPoint:TestPoint_Pad_D1.0mm, symbol Connector:TestPoint
Connections:
- net at J4.A7 (D-), J4.B7 (D-), R2.1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: now also TP2.1
- net at J4.A6 (D+), J4.B6 (D+), R1.1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: now also TP1.1
Changed lines of the file:
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@@
     (company "Rasmus L.")
+  )
+  (junction (at 165.1 63.5) (diameter 0) (color 0 0 0 0)
+  )
+  (junction (at 170.18 63.5) (diameter 0) (color 0 0 0 0)
   )
   (junction (at 170.18 49.53) (diameter 0) (color 0 0 0 0)
@@
     (stroke (width 0) (type default) (color 0 0 0 0))
   )
+  (wire (pts (xy 165.1 63.5) (xy 165.1 66.04))
+    (stroke (width 0) (type default) (color 0 0 0 0))
+  )
   (wire (pts (xy 138.43 73.66) (xy 139.7 73.66))
     (stroke (width 0) (type default) (color 0 0 0 0))
@@
     (stroke (width 0) (type default) (color 0 0 0 0))
   )
+  (wire (pts (xy 170.18 63.5) (xy 170.18 66.04))
+    (stroke (width 0) (type default) (color 0 0 0 0))
+  )
   (wire (pts (xy 46.99 33.02) (xy 43.18 33.02))
     (stroke (width 0) (type default) (color 0 0 0 0))
@@
     (stroke (width 0) (type default) (color 0 0 0 0))
   )
-  (wire (pts (xy 165.1 57.15) (xy 165.1 66.04))
+  (wire (pts (xy 165.1 57.15) (xy 165.1 63.5))
     (stroke (width 0) (type default) (color 0 0 0 0))
   )
@@
     (stroke (width 0) (type default) (color 0 0 0 0))
   )
-  (wire (pts (xy 170.18 49.53) (xy 170.18 66.04))
+  (wire (pts (xy 170.18 49.53) (xy 170.18 63.5))
     (stroke (width 0) (type default) (color 0 0 0 0))
   )
@@
     (pin "1")
   )
+  (symbol (lib_id "Connector:TestPoint") (at 165.1 63.5 90) (unit 1)
+    (in_bom yes) (on_board yes)
+    (property "Reference" "TP1" (id 0) (at 156.21 62.23 90))
+    (property "Value" "TestPoint" (id 1) (at 156.21 64.77 90))
+    (property "Footprint" "TestPoint:TestPoint_Pad_D1.0mm" (id 2) (at 165.1 58.42 0)
+      (effects (font (size 1.27 1.27)) hide)
+    )
+    (property "Datasheet" "~" (id 3) (at 165.1 58.42 0)
+      (effects (font (size 1.27 1.27)) hide)
+    )
+    (pin "1")
+  )
   (symbol (lib_id "power:GND") (at 78.74 34.29 0) (unit 1)
     (in_bom yes) (on_board yes)
@@
   (symbol (lib_id "Device:Varistor") (at 160.02 57.15 270) (unit 1)
     (in_bom yes) (on_board yes)
-    (property "Reference" "RV2" (id 0) (at 157.48 60.96 90)
+    (property "Reference" "RV2" (id 0) (at 160.02 59.69 90)
       (effects (font (size 1.27 1.27)) (justify left))
     )
@@
     )
     (property "Datasheet" "" (id 3) (at 40.64 83.82 0)
+      (effects (font (size 1.27 1.27)) hide)
+    )
+    (pin "1")
+  )
+  (symbol (lib_id "Connector:TestPoint") (at 170.18 63.5 270) (unit 1)
+    (in_bom yes) (on_board yes)
+    (property "Reference" "TP2" (id 0) (at 176.53 63.5 90)
+      (effects (font (size 1.27 1.27)) (justify left))
+    )
+    (property "Value" "TestPoint" (id 1) (at 173.99 66.04 90)
+      (effects (font (size 1.27 1.27)) (justify left))
+    )
+    (property "Footprint" "TestPoint:TestPoint_Pad_D1.0mm" (id 2) (at 170.18 68.58 0)
+      (effects (font (size 1.27 1.27)) hide)
+    )
+    (property "Datasheet" "~" (id 3) (at 170.18 68.58 0)
       (effects (font (size 1.27 1.27)) hide)
     )
@@
       (reference "RV2") (unit 1) (value "ESD protection varistor") (footprint "Resistor_SMD:R_0402_1005Metric")
     )
+    (path "/50fb6bd6-6721-48c6-8d81-be63cc58cbe7"
+      (reference "TP1") (unit 1) (value "TestPoint") (footprint "TestPoint:TestPoint_Pad_D1.0mm")
+    )
+    (path "/b7c27b12-2a9e-4630-a53a-4fe3dc54641a"
+      (reference "TP2") (unit 1) (value "TestPoint") (footprint "TestPoint:TestPoint_Pad_D1.0mm")
+    )
     (path "/e5a34e74-740d-4f11-ae22-b442e9a04463"

Commit message: recommit
Parts:
- removed D1: Diode, Diode_SMD:D_0402_1005Metric, symbol Device:D_Small
- removed FB1: Ferrite bead low-pass filter, Resistor_SMD:R_0402_1005Metric, symbol Device:FerriteBead_Small
- added R9: 5,1kΩ, Resistor_SMD:R_0402_1005Metric, symbol Device:R_Small
Connections:
- net +5V: now also R9.1
- net at C2.2, U1.24 (AVCC), U1.44 (AVCC): now also R9.2
Other:
- moved on the sheet: R6

Commit message: initial
Parts:
- removed C1, C7: 100nf, Capacitor_SMD:C_0402_1005Metric, symbol Device:C_Small
- removed R3: 10kΩ, Resistor_SMD:R_0402_1005Metric, symbol Device:R_Small
- added C10, C9: 100nF, Capacitor_SMD:C_0402_1005Metric, symbol Device:C_Small
- added D2: D_Schottky, DIY:SOD323_bättre, symbol Device:D_Schottky_Small
- added FB1: Ferrite, Resistor_SMD:R_0402_1005Metric, symbol Device:FerriteBead_Small
- added RV3: ESD protection varistor, Resistor_SMD:R_0402_1005Metric, symbol Device:Varistor
- C2: value 1µf -> 100nF
- C3, C4: value 22pf -> 100nF
- C5, C6: value 22pf -> 22pF
- C8: value 1µf -> 1µF
- R9: value 5,1kΩ -> 22Ω
- Y1: value Crystal_GND24_Small -> Crystal_GND24
- renumbered D2 to D1
Connections:
- net +5V: now also C10.1, C9.2, D2.1 (K); no longer F1.2
- net GND: now also C10.2, C9.1, RV3.1
- net at D1.2 (A): now also R8.2; no longer R8.1
- net at J4.A4 (VBUS), J4.A9 (VBUS), J4.B4 (VBUS)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: now also FB1.1, RV3.2; no longer F1.1
- net IO10 renamed D10
- net IO11 renamed D11
- net IO12 renamed D12
- net IO13 renamed D13
- net D13: now also R8.1; no longer R8.2
- net IO8 renamed D8
- net IO9 renamed D9
- new net: D2.2 (A), F1.2
- new net: F1.1, FB1.2
- no-connect marks 3 -> 5
Other:
- moved on the sheet: C2, C3, C4, C5, C6, C8, D1, F1, J1, J2, J3, J4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
