File: prod/epi.kicad_pcb (KiCad board)
At the start: 2 copper layers, 12.5 x 23.1 mm, 27 parts, among them J1 Conn_01x12, J2 Conn_01x12, J3 Conn_01x04, J4 USB_C_Receptacle_USB2.0, U1 ATmega32U4-M, Y1 16mhz

Commit message: slight redesign
Other:
- board size 12.5 x 23.1 mm -> 20 x 26.2 mm

Commit message: mostly readme
Other:
- board size 20 x 26.2 mm -> 20 x 26.1 mm
Changed lines of the file:
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@@
   (gr_line (start 100.087712 53.765671) (end 100.090416 53.768601) (layer "B.SilkS") (width 0.18))
   (gr_rect (start 99.25 56.5) (end 101.25 58.1) (layer "Dwgs.User") (width 0.2) (fill none))
-  (gr_line (start 106.25 36.3) (end 106.25 38.8) (layer "Edge.Cuts") (width 0.1))
-  (gr_line (start 93.75 36.3) (end 93.75 38.8) (layer "Edge.Cuts") (width 0.1))
-  (gr_line (start 110 40.8) (end 106.25 40.8) (layer "Edge.Cuts") (width 0.1))
+  (gr_line (start 110 36.4) (end 110 40.8) (layer "Edge.Cuts") (width 0.1))
+  (gr_arc (start 106.25 38.8) (mid 107.25 39.8) (end 106.25 40.8) (layer "Edge.Cuts") (width 0.1))
+  (gr_line (start 90 36.4) (end 90 40.8) (layer "Edge.Cuts") (width 0.1))
   (gr_line (start 95.3 42.7) (end 96.5 42.2) (layer "Edge.Cuts") (width 0.1))
-  (gr_line (start 90 40.8) (end 93.75 40.8) (layer "Edge.Cuts") (width 0.1))
+  (gr_arc (start 93.75 40.8) (mid 92.75 39.8) (end 93.75 38.8) (layer "Edge.Cuts") (width 0.1))
   (gr_line (start 96.5 42.2) (end 103.5 42.2) (layer "Edge.Cuts") (width 0.1))
   (gr_arc (start 106.25 40.8) (mid 105.25 39.8) (end 106.25 38.8) (layer "Edge.Cuts") (width 0.1))
   (gr_arc (start 93.75 38.8) (mid 94.75 39.8) (end 93.75 40.8) (layer "Edge.Cuts") (width 0.1))
-  (gr_line (start 104.7 36.3) (end 106.25 36.3) (layer "Edge.Cuts") (width 0.1))
-  (gr_line (start 104.7 42.7) (end 104.7 36.3) (layer "Edge.Cuts") (width 0.1))
+  (gr_line (start 104.7 36.4) (end 110 36.4) (layer "Edge.Cuts") (width 0.1))
+  (gr_line (start 104.7 42.7) (end 104.7 36.4) (layer "Edge.Cuts") (width 0.1))
   (gr_line (start 110 62.5) (end 110 40.8) (layer "Edge.Cuts") (width 0.1))
   (gr_line (start 90 62.5) (end 110 62.5) (layer "Edge.Cuts") (width 0.1))
   (gr_line (start 90 40.8) (end 90 62.5) (layer "Edge.Cuts") (width 0.1))
-  (gr_line (start 93.75 36.3) (end 95.3 36.3) (layer "Edge.Cuts") (width 0.1))
-  (gr_line (start 95.3 36.3) (end 95.3 42.7) (layer "Edge.Cuts") (width 0.1))
+  (gr_line (start 90 36.4) (end 95.3 36.4) (layer "Edge.Cuts") (width 0.1))
+  (gr_line (start 95.3 36.4) (end 95.3 42.7) (layer "Edge.Cuts") (width 0.1))
   (gr_line (start 103.5 42.2) (end 104.7 42.7) (layer "Edge.Cuts") (width 0.1))
   (gr_text "A1" (at 104.638095 51.943) (layer "B.SilkS")
